File: pcb/adelheid-xt.kicad_sch (KiCad schematic)
At the start: 211 parts, among them J1 OLED, U1 YAAJ_WeAct_BlackPill_Part_Lik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

Commit message: Finalize gerbers
Parts:
- added R1: 10K, Resistor_SMD:R_0805_2012Metric_Pad1.15x1.40mm_HandSolder, symbol Device:R
- added RST1: SW_Push, Buttons_Switches_SMD:SW_SPST_TL3342, symbol Switch:SW_Push
Connections:
- net COL0: now also U1.1 (PB12); no longer U1.35 (PB1)
- net COL1: now also U1.37 (PB10); no longer U1.34 (PB0)
- net COL10: now also U1.33 (PA7); no longer U1.2 (PB13)
- net COL11: now also U1.32 (PA6); no longer U1.1 (PB12)
- net COL2: now also U1.3 (PB14); no longer U1.33 (PA7)
- net COL3: now also U1.10 (PA15); no longer U1.28 (PA2)
- net COL4: now also U1.11 (PB3); no longer U1.27 (PA1)
- net COL5: now also U1.12 (PB4); no longer U1.26 (PA0)
- net COL6: now also U1.13 (PB5); no longer U1.24 (PC15)
- net COL7: now also U1.2 (PB13); no longer U1.37 (PB10)
- net COL9: now also U1.24 (PC15); no longer U1.3 (PB14)
- net GND: now also RST1.1
- net RA: now also U1.35 (PB1); no longer U1.31 (PA5)
- net RB: now also U1.34 (PB0); no longer U1.32 (PA6)
- net ROW0: now also U1.4 (PB15); no longer U1.30 (PA4)
- net ROW1: now also U1.16 (PB8); no longer U1.43 (SWIO)
- net ROW10: now also U1.28 (PA2); no longer U1.11 (PB3)
- net ROW11: now also U1.30 (PA4); no longer U1.5 (PA8)
- net ROW2: now also U1.27 (PA1); no longer U1.12 (PB4)
- net ROW3: now also U1.42 (SWCLK); no longer U1.17 (PB9)
- net ROW4: now also U1.29 (PA3); no longer U1.10 (PA15)
- net ROW5: now also U1.31 (PA5); no longer U1.4 (PB15)
- net ROW6: now also U1.5 (PA8); no longer U1.29 (PA3)
- net ROW7: now also U1.17 (PB9); no longer U1.42 (SWCLK)
- net ROW8: now also U1.26 (PA0); no longer U1.13 (PB5)
- net ROW9: now also U1.43 (SWIO); no longer U1.16 (PB8)
- net VCC: now also R1.1
- net RESET: now reaches U1.25 (RES)
- net RESET: now also R1.2, RST1.2
- no-connect marks 15 -> 14
Other:
- moved on the sheet: U1
